Commit message: Alpha version trying to start Gen3 with hexagons, IMU and cameras

File: kortex_description/arms/gen3/7dof/urdf/gen3_macro.xacro (robot description, xacro)
@@ -29,4 +29,5 @@
       <inertial>
         <origin xyz="-2.3E-05 -0.010364 -0.07336" rpy="0 0 0" />
+        <!--origin xyz="-2.3E-05 -0.010364 -0.1" rpy="0 0 0" /-->
         <mass value="1.3773" />
         <inertia ixx="0.00457" ixy="1E-06" ixz="2E-06" iyy="0.004831" iyz="0.000448" izz="0.001409" />
@@ -329,4 +330,145 @@
         <child  link="${prefix}camera_color_frame" />
       </joint>
+      <link name="${prefix}imu_link" />
+      <joint name="${prefix}imu_module" type="fixed">
+        <origin xyz="0 0.05639 -0.00305" rpy="3.14159265358979 3.14159265358979 0" />
+        <parent link="${prefix}end_effector_link" />
+        <child  link="${prefix}imu_link" />
+      </joint>
+    <gazebo reference="${prefix}camera_color_frame">
+      <sensor name="camera_rgb" type="camera">
+        <!--pose degrees="true">0 0 0 0 0 -90</pose-->
+        <!-- 20 cm between cameras: pose degrees="true">-0.15 0.0 0.0 0 0 -90</pose-->
+	<!-- 10 cm between cameras -->
+        <!--pose>-0.05 0.0 0.0 0 0 -90</pose-->
+        <!--pose>0.032 -0.03 0.0 0 0 4.71</pose-->
+        <!--pose>0.075 -0.03 0.0 0 0 4.71</pose-->
+        <pose>0.0 0.0 0.0   0.0 -1.5708 0.0</pose>
+        <visualize>true</visualize>
+        <update_rate>4</update_rate>
+        <!--always_on>1</always_on-->
+        <camera name="camera_rgb">
+          <!-- zoom cameras horizontal_fov>0.8</horizontal_fov -->
+          <!--pose>-0.25 0.0 0.0 0 0 0</pose-->
+          <!--horizontal_fov>1.21126</horizontal_fov-->
+          <horizontal_fov>1.0472</horizontal_fov>
+          <!--image_topic_name>image_raw</image_topic_name>
+          <camera_info_topic>camera_info</camera_info_topic-->
+          <image>
+            <width>1280</width>
+            <height>720</height>
+            <format>RGB_INT8</format>
+          </image>
+          <clip>
+            <near>0.001</near>
+            <far>25</far>
+          </clip>
+          <!--lens>
+            <intrinsics>
+              <fx>100</fx>
+              <fy>100</fy>
+              <cx>420</cx>
+              <cy>240</cy>
+              <s>0</s>
+            </intrinsics>
+          </lens-->
+        </camera>
+        <plugin name="camera_rgb_controller" filename="libgazebo_ros_camera.so">
+            <alwaysOn>true</alwaysOn>
+            <updateRate>4.0</updateRate>
+            <cameraName>realsense/camera_rgb</cameraName>
+            <imageTopicName>image_raw</imageTopicName>
+            <cameraInfoTopicName>camera_info</cameraInfoTopicName>
+            <frameName>${prefix}camera_color_frame</frameName>
+            <!--frame_name>camera_link</frame_name>
+                <always_on>true</always_on>
+            <update_rate>0.0</update_rate>
+            <camera_name>/realsense/camera_right</camera_name>
+            <image_topic_name>image_raw</image_topic_name>
+            <camera_info_topic_name>camera_info</camera_info_topic_name-->
+            <hackBaseline>0.4</hackBaseline>
+            <distortionK1>0.0</distortionK1>
+            <distortionK2>0.0</distortionK2>
+            <distortionK3>0.0</distortionK3>
+            <distortionT1>0.0</distortionT1>
+            <distortionT2>0.0</distortionT2>
+        </plugin>
+      </sensor>
+    </gazebo>
+    <gazebo reference="${prefix}camera_depth_frame">
+      <sensor name="camera_depth" type="depth">
+        <pose>0.0 0.0 0.0   0.0 -1.5708 0.0</pose>
+        <visualize>false</visualize>
+        <update_rate>4</update_rate>
+        <!--always_on>1</always_on-->
+        <camera name="camera_depth">
+          <!-- zoom cameras horizontal_fov>0.8</horizontal_fov -->
+          <!--pose>-0.25 0.0 0.0 0 0 0</pose-->
+          <!--horizontal_fov>1.21126</horizontal_fov-->
+          <horizontal_fov>1.0472</horizontal_fov>
+          <!--image_topic_name>image_raw</image_topic_name>
+          <camera_info_topic>camera_info</camera_info_topic-->
+          <image>
+            <width>424</width>
+            <height>240</height>
+            <!--format>RGB_INT8</format-->
+          </image>
+          <clip>
+            <near>0.001</near>
+            <far>25</far>
+          </clip>
+          <!--lens>
+            <intrinsics>
+              <fx>100</fx>
+              <fy>100</fy>
+              <cx>420</cx>
+              <cy>240</cy>
+              <s>0</s>
+            </intrinsics>
+          </lens-->
+        </camera>
+        <plugin name="camera_depth_controller" filename="libgazebo_ros_depth_camera.so">
+            <alwaysOn>true</alwaysOn>
+            <updateRate>4.0</updateRate>
+            <cameraName>realsense/camera_depth</cameraName>
+            <!--imageTopicName>image_raw</imageTopicName>
+            <cameraInfoTopicName>camera_info</cameraInfoTopicName-->
+            <depthImageTopicName>depth_raw</depthImageTopicName>
+            <depthImageCameraInfoTopicName>depth_info</depthImageCameraInfoTopicName>
+            <frameName>${prefix}camera_depth_frame</frameName>
+            <!--frame_name>camera_link</frame_name>
+                <always_on>true</always_on>
+            <update_rate>0.0</update_rate>
+            <camera_name>/realsense/camera_right</camera_name>
+            <image_topic_name>image_raw</image_topic_name>
+            <camera_info_topic_name>camera_info</camera_info_topic_name-->
+            <hackBaseline>0.55</hackBaseline>
+            <distortionK1>0.0</distortionK1>
+            <distortionK2>0.0</distortionK2>
+            <distortionK3>0.0</distortionK3>
+            <distortionT1>0.0</distortionT1>
+            <distortionT2>0.0</distortionT2>
+        </plugin>
+      </sensor>
+    </gazebo>
+    <gazebo reference="imu_link">
+      <gravity>true</gravity>
+      <sensor name="imu_sensor" type="imu">
+        <pose>0.0 0.0 0.0   0.0 -1.5708 0.0</pose>
+        <visualize>false</visualize>
+        <update_rate>8</update_rate>
+        <always_on>1</always_on>
+        <plugin name="imu_controller" filename="libgazebo_ros_imu_sensor.so">
+            <topicName>imu</topicName>
+            <bodyName>imu_link</bodyName>
+            <alwaysOn>true</alwaysOn>
+            <updateRateHZ>8</updateRateHZ>
+            <frameName>imu_link</frameName>
+            <gaussianNoise>0.0</gaussianNoise>
+            <xyzOffset>0 0 0</xyzOffset>
+            <rpyOffset>0 0 0</rpyOffset>
+        </plugin>
+      </sensor>
+    </gazebo>
     </xacro:if>
   </xacro:macro>

Commit message: Adjust cameras and robot's position, try to not start trajectory controller

File: kortex_description/arms/gen3/7dof/urdf/gen3_macro.xacro (robot description, xacro)
@@ -95,5 +95,5 @@
       <axis
         xyz="0 0 1" />
-      <limit lower="-2.24" upper="2.24" effort="39" velocity="1.3963" />
+      <limit lower="-2.25" upper="2.25" effort="39" velocity="1.3963" />
     </joint>
     <link name="${prefix}half_arm_2_link">
@@ -235,5 +235,5 @@
       <axis
         xyz="0 0 1" />
-      <limit lower="-2.09" upper="2.09" effort="9" velocity="1.2218" />
+      <limit lower="-2.1" upper="2.1" effort="9" velocity="1.2218" />
     </joint>
     <xacro:if value="${vision}">
@@ -312,13 +312,14 @@
     </joint>
     <xacro:if value="${vision}">
-      <link name="${prefix}camera_link" />
+      <!--link name="${prefix}camera_link" />
       <joint name="${prefix}camera_module" type="fixed">
         <origin xyz="0 0.05639 -0.00305" rpy="3.14159265358979 3.14159265358979 0" />
         <parent link="${prefix}end_effector_link" />
         <child  link="${prefix}camera_link" />
-      </joint>
+      </joint-->
       <link name="${prefix}camera_depth_frame" />
       <joint name="${prefix}depth_module" type="fixed">
-        <origin xyz="0.0275 0.066 -0.00305" rpy="3.14159265358979 3.14159265358979 0" />
+        <!--origin xyz="0.0275 0.066 -0.00305" rpy="3.14159265358979 3.14159265358979 0" /-->
+        <origin xyz="0.0275 0.066 0.00" rpy="3.14159265358979 3.14159265358979 1.5708" />
         <parent link="${prefix}end_effector_link" />
         <child  link="${prefix}camera_depth_frame" />
@@ -326,5 +327,5 @@
       <link name="${prefix}camera_color_frame" />
       <joint name="${prefix}color_module" type="fixed">
-        <origin xyz="0 0.05639 -0.00305" rpy="3.14159265358979 3.14159265358979 0" />
+        <origin xyz="0 0.05639 0.00" rpy="3.14159265358979 3.14159265358979 1.5708" />
         <parent link="${prefix}end_effector_link" />
         <child  link="${prefix}camera_color_frame" />
@@ -352,5 +353,6 @@
           <!--pose>-0.25 0.0 0.0 0 0 0</pose-->
           <!--horizontal_fov>1.21126</horizontal_fov-->
-          <horizontal_fov>1.0472</horizontal_fov>
+          <horizontal_fov>1.0472</horizontal_fov> <!-- 1.0472 is 60 degrees -->
+          <!--horizontal_fov>0.932</horizontal_fov--> <!-- camera is 60 degrees FOV diagonal, 16:9, thus 53.4 FOV horizontal -->
           <!--image_topic_name>image_raw</image_topic_name>
           <camera_info_topic>camera_info</camera_info_topic-->
@@ -406,5 +408,6 @@
           <!--pose>-0.25 0.0 0.0 0 0 0</pose-->
           <!--horizontal_fov>1.21126</horizontal_fov-->
-          <horizontal_fov>1.0472</horizontal_fov>
+          <!--horizontal_fov>1.0472</horizontal_fov-->
+          <horizontal_fov>1.129</horizontal_fov>
           <!--image_topic_name>image_raw</image_topic_name>
           <camera_info_topic>camera_info</camera_info_topic-->
@@ -436,4 +439,5 @@
             <depthImageTopicName>depth_raw</depthImageTopicName>
             <depthImageCameraInfoTopicName>depth_info</depthImageCameraInfoTopicName>
+            <pointCloudTopicName>depth</pointCloudTopicName>
             <frameName>${prefix}camera_depth_frame</frameName>
             <!--frame_name>camera_link</frame_name>

Commit message: less jitter when arm moves, correced X position in gazebo

File: kortex_description/arms/gen3/7dof/urdf/gen3_macro.xacro (robot description, xacro)
@@ -7,5 +7,5 @@
         <inertial>
           <origin xyz="-0.000648 -0.000166 0.084487" rpy="0 0 0" />
-          <mass value="1.697" />
+          <mass value="0.1697" />
           <inertia ixx="0.004622" ixy="9E-06" ixz="6E-05" iyy="0.004495" iyz="9E-06" izz="0.002079" />
         </inertial>
@@ -30,5 +30,5 @@
         <origin xyz="-2.3E-05 -0.010364 -0.07336" rpy="0 0 0" />
         <!--origin xyz="-2.3E-05 -0.010364 -0.1" rpy="0 0 0" /-->
-        <mass value="1.3773" />
+        <mass value="0.013773" />
         <inertia ixx="0.00457" ixy="1E-06" ixz="2E-06" iyy="0.004831" iyz="0.000448" izz="0.001409" />
       </inertial>
@@ -66,5 +66,5 @@
       <inertial>
         <origin xyz="-4.4E-05 -0.09958 -0.013278" rpy="0 0 0" />
-        <mass value="1.1636" />
+        <mass value="0.011636" />
         <inertia ixx="0.011088" ixy="5E-06" ixz="0" iyy="0.001072" iyz="-0.000691" izz="0.011255" />
       </inertial>
@@ -100,5 +100,5 @@
       <inertial>
         <origin xyz="-4.4E-05 -0.006641 -0.117892" rpy="0 0 0" />
-        <mass value="1.1636" />
+        <mass value="0.011636" />
         <inertia ixx="0.010932" ixy="0" ixz="-7E-06" iyy="0.011127" iyz="0.000606" izz="0.001043" />
       </inertial>
@@ -136,5 +136,5 @@
       <inertial>
         <origin xyz="-1.8E-05 -0.075478 -0.015006" rpy="0 0 0" />
-        <mass value="0.9302" />
+        <mass value="0.09302" />
         <inertia ixx="0.008147" ixy="-1E-06" ixz="0" iyy="0.000631" iyz="-0.0005" izz="0.008316" />
       </inertial>
@@ -170,5 +170,5 @@
       <inertial>
         <origin xyz="1E-06 -0.009432 -0.063883" rpy="0 0 0" />
-        <mass value="0.6781" />
+        <mass value="0.06781" />
         <inertia ixx="0.001596" ixy="0" ixz="0" iyy="0.001607" iyz="0.000256" izz="0.000399" />
       </inertial>
@@ -206,5 +206,5 @@
       <inertial>
         <origin xyz="1E-06 -0.045483 -0.00965" rpy="0 0 0" />
-        <mass value="0.6781" />
+        <mass value="0.06781" />
         <inertia ixx="0.001641" ixy="0" ixz="0" iyy="0.00041" iyz="-0.000278" izz="0.001641" />
       </inertial>
@@ -241,5 +241,5 @@
       <inertial>
         <origin xyz="0.000281 0.011402 -0.029798" rpy="0 0 0" />
-        <mass value="0.5" />
+        <mass value="0.05" />
         <inertia ixx="0.000587" ixy="3E-06" ixz="3E-06" iyy="0.000369" iyz="-0.000118" izz="0.000609" />
       </inertial>
@@ -265,5 +265,5 @@
       <inertial>
         <origin xyz="-9.3E-05 0.000132 -0.022905" rpy="0 0 0" />
-        <mass value="0.364" />
+        <mass value="0.0364" />
         <inertia ixx="0.000214" ixy="0" ixz="1E-06" iyy="0.000223" iyz="-2E-06" izz="0.00024" />
       </inertial>
