Commit message: First working version with husky and kortex

File: kortex_description/robots/husky_gen3_robotiq_2f_85.xacro (robot description, xacro)
@@ -1,12 +1,32 @@
 <?xml version="1.0"?>
 <robot name="gen3_robotiq_2f_85" xmlns:xacro="http://ros.org/wiki/xacro">
-    <!-- Arguments -->
+    <!-- Husky -->
+    <xacro:arg name="laser_enabled" default="false" />
+    <xacro:arg name="ur5_enabled" default="false" />
+    <xacro:arg name="kinect_enabled" default="false" />
+    <xacro:include filename="$(find husky_description)/urdf/husky.urdf.xacro"/>
+    <xacro:include filename="$(find husky_gazebo)/urdf/husky.gazebo.xacro" />
+    <!-- Gazebo plugin for ROS Control -->
+    <!--gazebo>
+      <plugin name="gazebo_ros_control" filename="libgazebo_ros_control.so">
+        <robotNamespace>my_gen3</robotNamespace>
+      </plugin>
+    </gazebo-->
+    <!--xacro:husky_robot /-->
+    <xacro:husky_robot_gazebo />
+    <!-- Gen3 -->
     <xacro:arg name="arm" default="gen3" />
     <xacro:arg name="dof" default="7" />
     <xacro:arg name="vision" default="true" />
     <xacro:arg name="gripper" default="robotiq_2f_85" />
+    <xacro:arg name="sim" default="false" />
     <xacro:arg name="prefix" default="" />
     <xacro:include filename="$(find kortex_description)/robots/husky_kortex_robot.xacro" />
-    <xacro:load_robot arm="$(arg arm)" gripper="$(arg gripper)" dof="$(arg dof)" vision="$(arg vision)" prefix="$(arg prefix)" />
+    <xacro:load_robot arm="$(arg arm)" gripper="$(arg gripper)" dof="$(arg dof)" vision="$(arg vision)" sim="$(arg sim)" prefix="$(arg prefix)" />
+    <joint name="husky_arm" type="fixed">
+      <parent link="top_plate_link" />
+      <child link="$(arg prefix)base_link" />
+      <origin xyz="0.2206 0 0" rpy="0 0 0" />
+    </joint>
     <!--xacro:include filename="$(find kortex_description)/launch/world_xy.xacro"/>
     <xacro:model_kinova reach="0.90"/-->

File: kortex_description/robots/husky_kortex_robot.xacro (robot description, xacro)
@@ -1,5 +1,5 @@
 <?xml version="1.0"?>
-<robot name="kinova_arm" xmlns:xacro="http://ros.org/wiki/xacro">
-    <xacro:macro name="load_robot" params="arm gripper dof vision prefix">
+<robot xmlns:xacro="http://ros.org/wiki/xacro">
+    <xacro:macro name="load_robot" params="arm gripper dof vision sim prefix">
         <!-- Files to include -->
         <xacro:include filename="$(find kortex_description)/arms/${arm}/${dof}dof/urdf/${arm}_macro.xacro" />
@@ -7,4 +7,12 @@
             <xacro:include filename="$(find kortex_description)/grippers/${gripper}/urdf/${gripper}_macro.xacro" />
         </xacro:unless>
+        <xacro:if value="${sim}">
+            <!-- Arm transmission elements-->
+            <xacro:include filename="$(find kortex_description)/arms/${arm}/${dof}dof/urdf/${arm}_transmission_macro.xacro" />
+            <!-- Gripper transmission elements if there is a gripper-->
+            <xacro:unless value="${not gripper}">
+                <xacro:include filename="$(find kortex_description)/grippers/${gripper}/urdf/${gripper}_transmission_macro.xacro" />
+            </xacro:unless>
+        </xacro:if>
         <!-- Run the macros -->
         <!-- Load the arm -->
@@ -27,11 +35,16 @@
             </joint>
         </xacro:if>
-        <!-- Link gen3 with husky -->
-        <link name="husky_gen3" />
-        <joint name="husky_gen3_joint" type="fixed">
-          <child link="${prefix}base_link" />
-          <parent link="top_plate_link" />
-          <origin xyz="0 0 0" rpy="0 0 0" />
-        </joint>
+        <!-- Load the Gazebo transmissions and gazebo_ros_control plugin -->
+        <xacro:if value="${sim}">
+            <xacro:load_gazebo_arm_transmissions prefix="${prefix}"/>
+            <xacro:unless value="${not gripper}">
+                <xacro:load_gazebo_gripper_transmissions prefix="${prefix}"/>
+            </xacro:unless>
+            <gazebo>
+                <plugin name="gazebo_ros_control" filename="libgazebo_ros_control.so">
+                    <legacyModeNS>true</legacyModeNS>
+                </plugin>
+            </gazebo>
+        </xacro:if>
     </xacro:macro>
 </robot>

Commit message: Add hexagons (not affected by robot movement)

File: kortex_description/robots/husky_gen3_robotiq_2f_85.xacro (robot description, xacro)
@@ -27,7 +27,5 @@
       <parent link="top_plate_link" />
       <child link="$(arg prefix)base_link" />
-      <origin xyz="0.2206 0 0" rpy="0 0 0" />
+      <origin xyz="0.30 0 -0.02" rpy="0 0 0" />
     </joint>
-    <!--xacro:include filename="$(find kortex_description)/launch/world_xy.xacro"/>
-    <xacro:model_kinova reach="0.90"/-->
 </robot>

Commit message: modify arm location on platform

File: kortex_description/robots/husky_gen3_robotiq_2f_85.xacro (robot description, xacro)
@@ -27,5 +27,5 @@
       <parent link="top_plate_link" />
       <child link="$(arg prefix)base_link" />
-      <origin xyz="0.30 0 -0.02" rpy="0 0 0" />
+      <origin xyz="0.25 0 0.01" rpy="0 0 0" />
     </joint>
 </robot>
